File: NI6739_test.kicad_sch (KiCad schematic)
At the start: 33 parts, among them J1 2-5174225-5

Commit message: Add progress 240419
Parts:
- added J2: Conn_01x34_Pin_A, symbol Connector:Conn_01x34_Pin
- added J3: Conn_01x34_Pin_B, symbol Connector:Conn_01x34_Pin
- C1, C10, C11, C12, C13, C14, C15, C16, C17, C18, C19, C2, C20, C21, C22, C23, C24, C25, C26, C27, C28, C29, C3, C30, C31, C32, C4, C5, C6, C7, C8, C9: value 0.1 -> 0.1u
Connections:
- net GND: now also J1.A11, J1.A14, J1.A18, J1.A19, J1.A20, J1.A24, J1.A27, J1.A30, J1.A33, J1.B1, J1.B12, J1.B15, J1.B16, J1.B21, J1.B22, J1.B25, J1.B28, J1.B3, J1.B31, J1.B34, J1.B5, J1.B7, J1.B8, J1.B9
- net AO 21: now reaches C21.2
- net AO 21: now also J3.26 (Pin_26)
- net AO 5: now reaches C5.1
- net AO 5: now also J3.13 (Pin_13)
- net AO 28: now reaches C28.2
- net AO 12: now reaches C12.1
- net AO 12: now also J3.19 (Pin_19)
- net AO 13: now reaches C13.1
- net AO 13: now also J3.20 (Pin_20)
- net AO 10: now reaches C10.1
- net AO 10: now also J3.17 (Pin_17)
- net AO 24: now reaches C24.2
- net AO 24: now also J2.29 (Pin_29)
- net AO 14: now reaches C14.1
- net AO 14: now also J2.21 (Pin_21)
- net AO 26: now reaches C26.2
- net AO 9: now reaches C9.1
- net AO 9: now also J2.17 (Pin_17)
- net AO 29: now reaches C29.2
- net AO 25: now reaches C25.2
- net AO 25: now also J3.29 (Pin_29)
- net AO 23: now reaches C23.2
- net AO 23: now also J2.28 (Pin_28)
- net AO 20: now reaches C20.2
- net AO 20: now also J2.26 (Pin_26)
- net AO 3: now reaches C3.1
- net AO 3: now also J2.12 (Pin_12)
- net AO 8: now reaches C8.1
- net AO 8: now also J2.16 (Pin_16)
- net AO 4: now reaches C4.1
- net AO 4: now also J2.13 (Pin_13)
- net AO 0: now reaches C1.1
- net AO 0: now also J2.10 (Pin_10)
- net AO 19: now reaches C19.2
- net AO 19: now also J2.25 (Pin_25)
- net AO 30: now reaches C30.2
- net AO 31: now reaches C31.2
- net AO 7: now reaches C7.1
- net AO 7: now also J2.15 (Pin_15)
- net AO 27: now reaches C27.2
- net AO 2: now reaches C2.1
- net AO 2: now also J3.11 (Pin_11)
- net AO 32: now reaches C32.2
- net AO 15: now reaches C15.1
- net AO 15: now also J2.22 (Pin_22)
- net AO 16: now reaches C16.1
- net AO 16: now also J2.23 (Pin_23)
- net AO 17: now reaches C17.1
- net AO 17: now also J3.23 (Pin_23)
- net AO 22: now reaches C22.2
- net AO 22: now also J3.27 (Pin_27)
- net AO 6: now reaches C6.1
- net AO 6: now also J3.14 (Pin_14)
- net AO 11: now reaches C11.1
- net AO 11: now also J3.18 (Pin_18)
- net AO 18: now reaches C18.1
- net AO 18: now also J3.24 (Pin_24)
- new net AO 1: J3.10 (Pin_10)

Commit message: Add sch for measure each pin of NI6739 connector
Connections:
- net AO 32 is gone; now on net AO 31: C32.2
- net AO 1: now also C2.1
- net AO 10: now also C11.1; no longer C10.1
- net AO 11: now also C12.1; no longer C11.1
- net AO 12: now also C13.1; no longer C12.1
- net AO 13: now also C14.1; no longer C13.1
- net AO 14: now also C15.1; no longer C14.1
- net AO 15: now also C16.1; no longer C15.1
- net AO 16: now also C17.1; no longer C16.1
- net AO 17: now also C18.1; no longer C17.1
- net AO 18: now also C19.2; no longer C18.1
- net AO 19: now also C20.2; no longer C19.2
- net AO 2: now also C3.1; no longer C2.1
- net AO 20: now also C21.2; no longer C20.2
- net AO 21: now also C22.2; no longer C21.2
- net AO 22: now also C23.2; no longer C22.2
- net AO 23: now also C24.2; no longer C23.2
- net AO 24: now also C25.2; no longer C24.2
- net AO 25: now also C26.2; no longer C25.2
- net AO 26: now also C27.2, J3.30 (Pin_30); no longer C26.2
- net AO 27: now also C28.2, J2.31 (Pin_31); no longer C27.2
- net AO 28: now also C29.2, J2.32 (Pin_32); no longer C28.2
- net AO 29: now also C30.2, J3.32 (Pin_32); no longer C29.2
- net AO 3: now also C4.1; no longer C3.1
- net AO 30: now also C31.2, J3.33 (Pin_33); no longer C30.2
- net AO 31: now also J2.34 (Pin_34); no longer C31.2
- net AO 4: now also C5.1; no longer C4.1
- net AO 5: now also C6.1; no longer C5.1
- net AO 6: now also C7.1; no longer C6.1
- net AO 7: now also C8.1; no longer C7.1
- net AO 8: now also C9.1; no longer C8.1
- net AO 9: now also C10.1; no longer C9.1
- net GND renamed GNDA
- net GNDA: no longer J1.B1, J1.B2, J1.B3, J1.B5, J1.B7, J1.B8, J1.B9
- new net GNDD: J1.B1, J1.B2, J1.B3, J1.B5, J1.B7, J1.B8, J1.B9
- no-connect marks 0 -> 48

Commit message: Add footprint
Parts:
- C1, C10, C11, C12, C13, C14, C15, C16, C17, C18, C19, C2, C20, C21, C22, C23, C24, C25, C26, C27, C28, C29, C3, C30, C31, C32, C4, C5, C6, C7, C8, C9: footprint (none) -> Capacitor_SMD:C_0603_1608Metric
- J1: footprint 251742255 -> SamacSys_Parts:251742255
- J2, J3: footprint (none) -> Connector_PinHeader_1.00mm:PinHeader_1x34_P1.00mm_Vertical_SMD_Pin1Left
Connections:
- net +5V: now also J2.1 (Pin_1)
- no-connect marks 48 -> 47
Changed lines of the file:
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@@
   (junction (at 199.39 149.86) (diameter 0) (color 0 0 0 0)
   )
-  (no_connect (at 215.9 30.48))
   (no_connect (at 241.3 68.58))
   (no_connect (at 241.3 48.26))
@@
       (effects (font (size 1.27 1.27)))
     )
-    (property "Footprint" "251742255" (at 113.03 54.61 0)
+    (property "Footprint" "SamacSys_Parts:251742255" (at 113.03 54.61 0)
       (effects (font (size 1.27 1.27)) (justify left) hide)
     )
@@
       (effects (font (size 1.27 1.27)) (justify left))
     )
-    (property "Footprint" "" (at 171.45 39.6748 0)
+    (property "Footprint" "Capacitor_SMD:C_0603_1608Metric" (at 171.45 39.6748 0)
       (effects (font (size 1.27 1.27)) hide)
     )
@@
       (effects (font (size 1.27 1.27)))
     )
-    (property "Footprint" "" (at 44.45 51.1048 0)
+    (property "Footprint" "Capacitor_SMD:C_0603_1608Metric" (at 44.45 51.1048 0)
       (effects (font (size 1.27 1.27)) hide)
     )
@@
       (effects (font (size 1.27 1.27)))
     )
-    (property "Footprint" "" (at 171.45 114.6048 0)
+    (property "Footprint" "Capacitor_SMD:C_0603_1608Metric" (at 171.45 114.6048 0)
       (effects (font (size 1.27 1.27)) hide)
     )
@@
     )
   )
+  (symbol (lib_id "power:+5V") (at 215.9 30.48 270) (unit 1)
+    (in_bom yes) (on_board yes) (dnp no) (fields_autoplaced)
+    (property "Reference" "#PWR03" (at 212.09 30.48 0)
+      (effects (font (size 1.27 1.27)) hide)
+    )
+    (property "Value" "+5V" (at 219.71 30.48 90)
+      (effects (font (size 1.27 1.27)) (justify left))
+    )
+    (property "Footprint" "" (at 215.9 30.48 0)
+      (effects (font (size 1.27 1.27)) hide)
+    )
+    (property "Datasheet" "" (at 215.9 30.48 0)
+      (effects (font (size 1.27 1.27)) hide)
+    )
+    (pin "1")
+    (instances
+      (project "NI6739_test"
+        (path "/917f02e4-9203-46de-ad00-6541640ee35f"
+          (reference "#PWR03") (unit 1)
+        )
+      )
+    )
+  )
   (symbol (lib_id "Device:C") (at 40.64 128.27 90) (unit 1)
     (in_bom yes) (on_board yes) (dnp no) (fields_autoplaced)
@@
       (effects (font (size 1.27 1.27)))
     )
-    (property "Footprint" "" (at 44.45 127.3048 0)
+    (property "Footprint" "Capacitor_SMD:C_0603_1608Metric" (at 44.45 127.3048 0)
       (effects (font (size 1.27 1.27)) hide)
     )
@@
       (effects (font (size 1.27 1.27)))
     )
-    (property "Footprint" "" (at 44.45 138.7348 0)
+    (property "Footprint" "Capacitor_SMD:C_0603_1608Metric" (at 44.45 138.7348 0)
       (effects (font (size 1.27 1.27)) hide)
     )
@@
       (effects (font (size 1.27 1.27)))
     )
-    (property "Footprint" "" (at 44.45 104.4448 0)
+    (property "Footprint" "Capacitor_SMD:C_0603_1608Metric" (at 44.45 104.4448 0)
       (effects (font (size 1.27 1.27)) hide)
     )
@@
       (effects (font (size 1.27 1.27)))
     )
-    (property "Footprint" "" (at 171.45 73.9648 0)
+    (property "Footprint" "Capacitor_SMD:C_0603_1608Metric" (at 171.45 73.9648 0)
       (effects (font (size 1.27 1.27)) hide)
     )
@@
       (effects (font (size 1.27 1.27)))
     )
-    (property "Footprint" "" (at 44.45 148.8948 0)
+    (property "Footprint" "Capacitor_SMD:C_0603_1608Metric" (at 44.45 148.8948 0)
       (effects (font (size 1.27 1.27)) hide)
     )
@@
       (effects (font (size 1.27 1.27)))
     )
-    (property "Footprint" "" (at 171.45 94.2848 0)
+    (property "Footprint" "Capacitor_SMD:C_0603_1608Metric" (at 171.45 94.2848 0)
       (effects (font (size 1.27 1.27)) hide)
     )
@@
       (effects (font (size 1.27 1.27)))
     )
-    (property "Footprint" "" (at 44.45 95.5548 0)
+    (property "Footprint" "Capacitor_SMD:C_0603_1608Metric" (at 44.45 95.5548 0)
       (effects (font (size 1.27 1.27)) hide)
     )
@@
       (effects (font (size 1.27 1.27)))
     )
-    (property "Footprint" "" (at 171.45 126.0348 0)
+    (property "Footprint" "Capacitor_SMD:C_0603_1608Metric" (at 171.45 126.0348 0)
       (effects (font (size 1.27 1.27)) hide)
     )
@@
       (effects (font (size 1.27 1.27)))
     )
-    (property "Footprint" "" (at 171.45 85.3948 0)
+    (property "Footprint" "Capacitor_SMD:C_0603_1608Metric" (at 171.45 85.3948 0)
       (effects (font (size 1.27 1.27)) hide)
     )
@@
       (effects (font (size 1.27 1.27)))
     )
-    (property "Footprint" "" (at 171.45 61.2648 0)
+    (property "Footprint" "Capacitor_SMD:C_0603_1608Metric" (at 171.45 61.2648 0)
       (effects (font (size 1.27 1.27)) hide)
     )
@@
       (effects (font (size 1.27 1.27)))
     )
-    (property "Footprint" "" (at 171.45 33.3248 0)
+    (property "Footprint" "Capacitor_SMD:C_0603_1608Metric" (at 171.45 33.3248 0)
       (effects (font (size 1.27 1.27)) hide)
     )
@@
       (effects (font (size 1.27 1.27)))
     )
-    (property "Footprint" "" (at 44.45 34.5948 0)
+    (property "Footprint" "Capacitor_SMD:C_0603_1608Metric" (at 44.45 34.5948 0)
       (effects (font (size 1.27 1.27)) hide)
     )
@@
       (effects (font (size 1.27 1.27)))
     )
-    (property "Footprint" "" (at 44.45 86.6648 0)
+    (property "Footprint" "Capacitor_SMD:C_0603_1608Metric" (at 44.45 86.6648 0)
       (effects (font (size 1.27 1.27)) hide)
     )
@@
       (effects (font (size 1.27 1.27)) (justify left))
     )
-    (property "Footprint" "" (at 44.45 40.9448 0)
+    (property "Footprint" "Capacitor_SMD:C_0603_1608Metric" (at 44.45 40.9448 0)
       (effects (font (size 1.27 1.27)) hide)
     )
@@
       (effects (font (size 1.27 1.27)))
     )
-    (property "Footprint" "" (at 44.45 15.5448 0)
+    (property "Footprint" "Capacitor_SMD:C_0603_1608Metric" (at 44.45 15.5448 0)
       (effects (font (size 1.27 1.27)) hide)
     )
@@
       (effects (font (size 1.27 1.27)))
     )
-    (property "Footprint" "" (at 171.45 21.8948 0)
+    (property "Footprint" "Capacitor_SMD:C_0603_1608Metric" (at 171.45 21.8948 0)
       (effects (font (size 1.27 1.27)) hide)
     )
@@
       (effects (font (size 1.27 1.27)))
     )
-    (property "Footprint" "" (at 171.45 137.4648 0)
+    (property "Footprint" "Capacitor_SMD:C_0603_1608Metric" (at 171.45 137.4648 0)
       (effects (font (size 1.27 1.27)) hide)
     )
@@
       (effects (font (size 1.27 1.27)))
     )
-    (property "Footprint" "" (at 236.22 71.12 0)
+    (property "Footprint" "Connector_PinHeader_1.00mm:PinHeader_1x34_P1.00mm_Vertical_SMD_Pin1Left" (at 236.22 71.12 0)
       (effects (font (size 1.27 1.27)) hide)
     )
@@
       (effects (font (size 1.27 1.27)))
     )
-    (property "Footprint" "" (at 171.45 147.6248 0)
+    (property "Footprint" "Capacitor_SMD:C_0603_1608Metric" (at 171.45 147.6248 0)
       (effects (font (size 1.27 1.27)) hide)
     )
@@
       (effects (font (size 1.27 1.27)))
     )
-    (property "Footprint" "" (at 210.82 71.12 0)
+    (property "Footprint" "Connector_PinHeader_1.00mm:PinHeader_1x34_P1.00mm_Vertical_SMD_Pin1Left" (at 210.82 71.12 0)
       (effects (font (size 1.27 1.27)) hide)
     )
@@
       (effects (font (size 1.27 1.27)))
     )
-    (property "Footprint" "" (at 44.45 75.2348 0)
+    (property "Footprint" "Capacitor_SMD:C_0603_1608Metric" (at 44.45 75.2348 0)
       (effects (font (size 1.27 1.27)) hide)
     )
@@
       (effects (font (size 1.27 1.27)))
     )
-    (property "Footprint" "" (at 171.45 103.1748 0)
+    (property "Footprint" "Capacitor_SMD:C_0603_1608Metric" (at 171.45 103.1748 0)
       (effects (font (size 1.27 1.27)) hide)
     )
@@
       (effects (font (size 1.27 1.27)))
     )
-    (property "Footprint" "" (at 44.45 26.9748 0)
+    (property "Footprint" "Capacitor_SMD:C_0603_1608Metric" (at 44.45 26.9748 0)
       (effects (font (size 1.27 1.27)) hide)
     )
@@
       (effects (font (size 1.27 1.27)))
     )
-    (property "Footprint" "" (at 171.45 159.0548 0)
+    (property "Footprint" "Capacitor_SMD:C_0603_1608Metric" (at 171.45 159.0548 0)
       (effects (font (size 1.27 1.27)) hide)
     )
@@
       (effects (font (size 1.27 1.27)))
     )
-    (property "Footprint" "" (at 44.45 160.3248 0)
+    (property "Footprint" "Capacitor_SMD:C_0603_1608Metric" (at 44.45 160.3248 0)
       (effects (font (size 1.27 1.27)) hide)
     )
@@
       (effects (font (size 1.27 1.27)))
     )
-    (property "Footprint" "" (at 44.45 170.4848 0)
+    (property "Footprint" "Capacitor_SMD:C_0603_1608Metric" (at 44.45 170.4848 0)
       (effects (font (size 1.27 1.27)) hide)
     )
@@
       (effects (font (size 1.27 1.27)))
     )
-    (property "Footprint" "" (at 44.45 183.1848 0)
+    (property "Footprint" "Capacitor_SMD:C_0603_1608Metric" (at 44.45 183.1848 0)
       (effects (font (size 1.27 1.27)) hide)
     )
@@
       (effects (font (size 1.27 1.27)))
     )
-    (property "Footprint" "" (at 171.45 49.8348 0)
+    (property "Footprint" "Capacitor_SMD:C_0603_1608Metric" (at 171.45 49.8348 0)
       (effects (font (size 1.27 1.27)) hide)
     )
@@
       (effects (font (size 1.27 1.27)))
     )
-    (property "Footprint" "" (at 44.45 62.5348 0)
+    (property "Footprint" "Capacitor_SMD:C_0603_1608Metric" (at 44.45 62.5348 0)
       (effects (font (size 1.27 1.27)) hide)
     )
@@
       (effects (font (size 1.27 1.27)))
     )
-    (property "Footprint" "" (at 44.45 115.8748 0)
+    (property "Footprint" "Capacitor_SMD:C_0603_1608Metric" (at 44.45 115.8748 0)
       (effects (font (size 1.27 1.27)) hide)
     )
@@
       (effects (font (size 1.27 1.27)))
     )
-    (property "Footprint" "" (at 44.45 194.6148 0)
-      (effects (font (size 1.27 1.27)) hide)
-    )
+    (property "Footprint" "Capacitor_SMD:C_0603_1608Metric" (at 44.45 194.6148 0)
+      (effects (font (size 1.27 1.27)) hide)
+    )
